File: retropie-minicade-hat.kicad_pcb (KiCad board)
At the start: 4 copper layers, 65 x 32.7 mm, 17 parts, among them J1 40HAT, J2 Screw_Terminal_01x02, J3 Conn_02x02_Odd_Even, J4 Conn_02x02_Odd_Even, J5 Conn_01x08_Male, J6 Conn_01x08_Male, J7 Conn_01x03_Male, J8 Conn_02x03_Odd_Even, Q1 DMG2305UX, Q2 MMDT5401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

Commit message: change to C1 and C2 values
update to 22uF from 10uF in BOM.
No change to production files
Parts:
- C1, C2: value 10uF -> 22uF
Changed lines of the file:
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@@
   (net 34 "/SP_GPIO_7")
   (net 35 "/SP_GPIO_26")
-  (net 36 "Net-(R1-Pad1)")
+  (net 36 "Net-(Q2-Pad2)")
   (footprint "project_footprints:NPTH_3mm_ID" locked (layer "F.Cu")
     (at 82.04 64.31)
@@
     (fp_line (start 0.8 0.4125) (end -0.8 0.4125) (layer "F.Fab") (width 0.1))
     (pad "1" smd roundrect (at -0.825 0 270) (size 0.8 0.95) (layers "F.Cu" "F.Paste" "F.Mask") (roundrect_rratio 0.25)
-      (net 36 "Net-(R1-Pad1)") (pintype "passive"))
+      (net 36 "Net-(Q2-Pad2)") (pintype "passive"))
     (pad "2" smd roundrect (at 0.825 0 270) (size 0.8 0.95) (layers "F.Cu" "F.Paste" "F.Mask") (roundrect_rratio 0.25)
       (net 1 "GND") (pintype "passive"))
@@
       (effects (font (size 1 1) (thickness 0.15)))
     )
-    (fp_text value "10uF" (at 0 1.43) (layer "F.Fab")
+    (fp_text value "22uF" (at 0 1.43) (layer "F.Fab")
       (effects (font (size 1 1) (thickness 0.15)))
     )
@@
       (net 7 "/P5V") (pinfunction "E1") (pintype "passive"))
     (pad "2" smd rect (at -0.95 0 180) (size 0.65 0.4) (layers "F.Cu" "F.Paste" "F.Mask")
-      (net 36 "Net-(R1-Pad1)") (pinfunction "B1") (pintype "input"))
+      (net 36 "Net-(Q2-Pad2)") (pinfunction "B1") (pintype "input"))
     (pad "3" smd rect (at -0.95 0.65 180) (size 0.65 0.4) (layers "F.Cu" "F.Paste" "F.Mask")
       (net 6 "/P5V_HAT") (pinfunction "C2") (pintype "passive"))
@@
       (net 4 "Net-(Q1-Pad1)") (pinfunction "E2") (pintype "passive"))
     (pad "5" smd rect (at 0.95 0 180) (size 0.65 0.4) (layers "F.Cu" "F.Paste" "F.Mask")
-      (net 36 "Net-(R1-Pad1)") (pinfunction "B2") (pintype "input"))
+      (net 36 "Net-(Q2-Pad2)") (pinfunction "B2") (pintype "input"))
     (pad "6" smd rect (at 0.95 -0.65 180) (size 0.65 0.4) (layers "F.Cu" "F.Paste" "F.Mask")
-      (net 36 "Net-(R1-Pad1)") (pinfunction "C1") (pintype "passive"))
+      (net 36 "Net-(Q2-Pad2)") (pinfunction "C1") (pintype "passive"))
     (model "${KICAD6_3DMODEL_DIR}/Package_TO_SOT_SMD.3dshapes/SOT-363_SC-70-6.wrl"
       (offset (xyz 0 0 0))
@@
       (effects (font (size 1 1) (thickness 0.15)))
     )
-    (fp_text value "10uF" (at 0 1.43) (layer "F.Fab")
-      (effects (font (size 1 1) (thickness 0.15)))
-    )
+    (fp_text value "22uF" (at 0 1.43) (layer "F.Fab")
+      (effects (font (size 1 1) (thickness 0.15)))
+    )

Commit message: changed the H2G2 quote to something related to Hotblack
Other:
- board text added: "Hotblack Desiato: {dblquote}{dblquote} Hotblack's Minder: {dblquote}He's spending a year dead for tax purposes{dblquote}"
- board text removed: "This must be a Thursday. I never could get the hang of Thursdays!"
Changed lines of the file:
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@@
     (effects (font (size 0.9 0.9) (thickness 0.12)))
   )
-  (gr_text "This must be a Thursday. I never could get the hang of Thursdays!" (at 111.76 55.626) (layer "B.SilkS")
-    (effects (font (size 0.9 0.9) (thickness 0.12) italic) (justify mirror))
+  (gr_text "Hotblack Desiato: {dblquote}{dblquote}\nHotblack's Minder: {dblquote}He's spending a year dead for tax purposes{dblquote}" (at 135.001 54.991) (layer "B.SilkS")
+    (effects (font (size 0.9 0.9) (thickness 0.12) italic) (justify left mirror))
   )
   (gr_text "B3" (at 118.11 55.88 90) (layer "F.SilkS")
