File: retropie-minicade-hat.kicad_pcb (KiCad board)
At the start: 4 copper layers, 65 x 32.7 mm, 17 parts, among them J1 40HAT, J2 Screw_Terminal_01x02, J3 Conn_02x02_Odd_Even, J4 Conn_02x02_Odd_Even, J5 Conn_01x08_Male, J6 Conn_01x08_Male, J7 Conn_01x03_Male, J8 Conn_02x03_Odd_Even, Q1 DMG2305UX, Q2 MMDT5401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

Commit message: updated images and gerbers (Rev2)
updated gerbers to latest version of PCB
Other:
- board text added: "rev 2"
- board text removed: "rev 1"
