File: retropie-minicade-hat.kicad_sch (KiCad schematic)
At the start: 17 parts, among them J1 40HAT, J2 Screw_Terminal_01x02, J3 Conn_02x02_Odd_Even, J4 Conn_02x02_Odd_Even, J5 Conn_01x08_Male, J6 Conn_01x08_Male, J7 Conn_01x03_Male, J8 Conn_02x03_Odd_Even, Q1 DMG2305UX, Q2 MMDT5401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

Commit message: change to C1 and C2 values
update to 22uF from 10uF in BOM.
No change to production files
Parts:
- C1, C2: value 10uF -> 22uF
Changed lines of the file:
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@@
       (effects (font (size 1.27 1.27)) (justify left))
     )
-    (property "Value" "10uF" (id 1) (at 99.8839 138.1031 0)
+    (property "Value" "22uF" (id 1) (at 99.8839 138.1031 0)
       (effects (font (size 1.27 1.27)) (justify left))
     )
@@
       (effects (font (size 1.27 1.27)) (justify left))
     )
-    (property "Value" "10uF" (id 1) (at 70.1622 138.2298 0)
+    (property "Value" "22uF" (id 1) (at 70.1622 138.2298 0)
       (effects (font (size 1.27 1.27)) (justify left))
     )
@@
     )
     (path "/0388b81b-7bfb-4a23-9444-5dbf72eb6a1d"
-      (reference "C1") (unit 1) (value "10uF") (footprint "Capacitor_SMD:C_0603_1608Metric")
+      (reference "C1") (unit 1) (value "22uF") (footprint "Capacitor_SMD:C_0603_1608Metric")
     )
     (path "/3b43264c-4f36-4eb7-aaf5-1328e808310f"
-      (reference "C2") (unit 1) (value "10uF") (footprint "Capacitor_SMD:C_0603_1608Metric")
+      (reference "C2") (unit 1) (value "22uF") (footprint "Capacitor_SMD:C_0603_1608Metric")
     )
     (path "/00000000-0000-0000-0000-00005834bc4a"

Commit message: Update BOM with component numbers. ignore auto backups
Parts:
- C1, C2: LCSC Part # (none) -> C86295
- J1: LCSC Part # (none) -> C169819
- J2: LCSC Part # (none) -> C8404
- Q1: LCSC Part # (none) -> C150470
- Q2: LCSC Part # (none) -> C54540
- R1: LCSC Part # (none) -> C25804
- R2: LCSC Part # (none) -> C25819
- U1: LCSC Part # (none) -> C173386
Changed lines of the file:
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@@
     )
     (property "Datasheet" "" (id 3) (at 48.26 57.15 0))
+    (property "LCSC Part #" "C169819" (id 4) (at 66.04 57.15 0)
+      (effects (font (size 1.27 1.27)) hide)
+    )
     (pin "1")
     (pin "10")
@@
     )
     (property "Datasheet" "" (id 3) (at 156.21 60.96 0))
+    (property "LCSC Part #" "C150470" (id 4) (at 156.21 60.96 0)
+      (effects (font (size 1.27 1.27)) hide)
+    )
     (pin "1")
     (pin "2")
@@
       (effects (font (size 1.27 1.27)) hide)
     )
+    (property "LCSC Part #" "C25804" (id 4) (at 146.05 91.44 0)
+      (effects (font (size 1.27 1.27)) hide)
+    )
     (pin "1")
     (pin "2")
@@
       (effects (font (size 1.27 1.27)) hide)
     )
+    (property "LCSC Part #" "C25819" (id 4) (at 166.37 91.44 0)
+      (effects (font (size 1.27 1.27)) hide)
+    )
     (pin "1")
     (pin "2")
@@
     )
     (property "Datasheet" "~" (id 3) (at 97.5598 136.2302 0)
+      (effects (font (size 1.27 1.27)) hide)
+    )
+    (property "LCSC Part #" "C86295" (id 4) (at 97.5598 136.2302 0)
       (effects (font (size 1.27 1.27)) hide)
     )
@@
       (effects (font (size 1.27 1.27)) hide)
     )
+    (property "LCSC Part #" "C86295" (id 4) (at 67.8381 136.3569 0)
+      (effects (font (size 1.27 1.27)) hide)
+    )
     (pin "1")
     (pin "2")
@@
       (effects (font (size 1.27 1.27)) hide)
     )
+    (property "LCSC Part #" "C8404" (id 4) (at 129.54 63.5 0)
+      (effects (font (size 1.27 1.27)) hide)
+    )
     (pin "1")
     (pin "2")
@@
     )
     (property "Datasheet" "http://www.diodes.com/_files/datasheets/ds30169.pdf" (id 3) (at 148.5889 76.2445 0)
+      (effects (font (size 1.27 1.27)) hide)
+    )
+    (property "LCSC Part #" "C54540" (id 4) (at 148.5889 76.2445 0)
       (effects (font (size 1.27 1.27)) hide)
     )
@@
       (effects (font (size 1.27 1.27)) hide)
     )
+    (property "LCSC Part #" "C173386" (id 4) (at 83.0623 133.5898 0)
+      (effects (font (size 1.27 1.27)) hide)
+    )
     (pin "1")
     (pin "2")
@@
       (effects (font (size 1.27 1.27)) hide)
     )
+    (property "LCSC Part #" "C54540" (id 4) (at 163.83 76.2 0)
+      (effects (font (size 1.27 1.27)) hide)
+    )

Commit message: tweaks to pin order to rationalize trace routes
Connections:
- net BUTT_1: now also J5.4 (Pin_4); no longer J5.5 (Pin_5)
- net ENTER: now also J6.3 (Pin_3); no longer J6.2 (Pin_2)
- net JOY_DOWN: now also J5.6 (Pin_6); no longer J5.7 (Pin_7)
- net JOY_RIGHT: now also J5.7 (Pin_7); no longer J5.6 (Pin_6)
- net JOY_UP: now also J5.5 (Pin_5); no longer J5.4 (Pin_4)
- net PWR_BUTT: now also J6.2 (Pin_2); no longer J6.3 (Pin_3)
Changed lines of the file:
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@@
     (effects (font (size 1.27 1.27)) (justify left bottom))
   )
-  (label "JOY_DOWN" (at 167.4588 125.3537 0)
+  (label "JOY_DOWN" (at 167.4588 122.8137 0)
     (effects (font (size 1.27 1.27)) (justify left bottom))
   )
@@
     (effects (font (size 1.27 1.27)) (justify left bottom))
   )
-  (label "JOY_UP" (at 167.4588 117.7337 0)
+  (label "JOY_UP" (at 167.4588 120.2737 0)
     (effects (font (size 1.27 1.27)) (justify left bottom))
   )
@@
     (effects (font (size 1.27 1.27)) (justify left bottom))
   )
-  (label "JOY_RIGHT" (at 167.4588 122.8137 0)
+  (label "JOY_RIGHT" (at 167.4588 125.3537 0)
     (effects (font (size 1.27 1.27)) (justify left bottom))
   )
@@
     (effects (font (size 1.27 1.27)) (justify left bottom))
   )
-  (label "ENTER" (at 137.6383 112.8467 0)
+  (label "ENTER" (at 137.6383 115.3867 0)
     (effects (font (size 1.27 1.27)) (justify left bottom))
   )
@@
     (effects (font (size 1.27 1.27)) (justify left bottom))
   )
-  (label "PWR_BUTT" (at 137.6383 115.3867 0)
+  (label "PWR_BUTT" (at 137.6383 112.8467 0)
     (effects (font (size 1.27 1.27)) (justify left bottom))
   )
@@
     (effects (font (size 1.27 1.27)) (justify left bottom))
   )
-  (label "BUTT_1" (at 167.4588 120.2737 0)
+  (label "BUTT_1" (at 167.4588 117.7337 0)
     (effects (font (size 1.27 1.27)) (justify left bottom))
   )

Commit message: updated images and gerbers (Rev2)
updated gerbers to latest version of PCB
Parts:
- C1, C2: LCSC Part # C86295 -> C59461
- J2: footprint TerminalBlock:TerminalBlock_bornier-2_P5.08mm -> TerminalBlock_4Ucon:TerminalBlock_4Ucon_1x02_P3.50mm_Horizontal
- U1: LCSC Part # C173386 -> C6186
