File: 2-layer/retropie-hat-2L.kicad_pcb (KiCad board)
At the start: 2 copper layers, 65 x 32.7 mm, 17 parts, among them J1 40HAT, J2 Screw_Terminal_01x02, J3 Conn_02x02_Odd_Even, J4 Conn_02x02_Odd_Even, J5 Conn_01x08_Male, J6 Conn_01x08_Male, J7 Conn_01x03_Male, J8 Conn_02x03_Odd_Even, Q1 DMG2305UX, Q2 MMDT5401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

Commit message: updated images and gerbers (Rev2)
updated gerbers to latest version of PCB
Parts:
- J2: footprint TerminalBlock:TerminalBlock_bornier-2_P5.08mm -> TerminalBlock_4Ucon:TerminalBlock_4Ucon_1x02_P3.50mm_Horizontal
- moved R1 1.37 mm to (88.0, 77.3), turned to 180 degrees
- moved R2 1.36 mm to (88.0, 75.8), turned to 0 degrees
- moved J2 1.36 mm to (81.7, 74.0)
- moved J5 0.12 mm to (115.1, 58.0)
Routing:
- net Net-(Q2A-B1): track 6.26 -> 8.25 mm
- net Net-(Q1-G): track 6.46 -> 6.97 mm
Other:
- board size 65 x 32.7 mm -> 65 x 32.3 mm
- board text added: "rev 2"
- board text removed: "rev 1"
