File: 2-layer/retropie-hat-2L.kicad_sch (KiCad schematic)
At the start: 0 parts

Commit message: updated images and gerbers (Rev2)
updated gerbers to latest version of PCB
Other:
- sheet base sheet: file ..\retropie-minicade-hat.kicad_sch -> ../retropie-minicade-hat.kicad_sch
Changed lines of the file:
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@@
-(kicad_sch (version 20211123) (generator eeschema)
+(kicad_sch (version 20230121) (generator eeschema)
   (paper "A4")
   (sheet (at 74.7808 50.9992) (size 58.0612 43.2348) (fields_autoplaced)
-    (stroke (width 0.1524) (type solid) (color 0 0 0 0))
+    (stroke (width 0.1524) (type solid))
     (fill (color 0 0 0 0.0000))
-    (property "Sheet name" "base sheet" (id 0) (at 74.7808 50.2876 0)
+    (property "Sheetname" "base sheet" (at 74.7808 50.2876 0)
       (effects (font (size 1.27 1.27)) (justify left bottom))
     )
-    (property "Sheet file" "..\\retropie-minicade-hat.kicad_sch" (id 1) (at 74.7808 94.8186 0)
+    (property "Sheetfile" "../retropie-minicade-hat.kicad_sch" (at 74.7808 94.8186 0)
       (effects (font (size 1.27 1.27)) (justify left top))
+    )
+    (instances
+      (project "retropie-hat-2L"
+        (path "/f16a6529-34cc-45d3-b796-fa1b9f3df7d3" (page "2"))
+      )
     )
   )
   (sheet_instances
     (path "/" (page "1"))
-    (path "/f24b66b4-45fc-4e7b-bc4d-d13b5ccb77d9" (page "2"))
-  )
-  (symbol_instances
-    (path "/f24b66b4-45fc-4e7b-bc4d-d13b5ccb77d9/cb052714-d958-4db1-ac69-e78f6bdf079a"
-      (reference "#PWR01") (unit 1) (value "GND") (footprint "")
-    )
-    (path "/f24b66b4-45fc-4e7b-bc4d-d13b5ccb77d9/00000000-0000-0000-0000-000058e15a41"
-      (reference "#PWR02") (unit 1) (value "GND") (footprint "")
-    )
-    (path "/f24b66b4-45fc-4e7b-bc4d-d13b5ccb77d9/00000000-0000-0000-0000-000058e15a9e"
-      (reference "#PWR03") (unit 1) (value "GND") (footprint "")
-    )
-    (path "/f24b66b4-45fc-4e7b-bc4d-d13b5ccb77d9/d00fc5d3-1591-436f-8a72-4f878c3cfed0"
-      (reference "#PWR04") (unit 1) (value "GND") (footprint "")
-    )
-    (path "/f24b66b4-45fc-4e7b-bc4d-d13b5ccb77d9/2d0c4002-e7ff-4076-abe4-93ece123726b"
-      (reference "#PWR05") (unit 1) (value "GND") (footprint "")
-    )
-    (path "/f24b66b4-45fc-4e7b-bc4d-d13b5ccb77d9/000b27f2-f926-40dc-af69-bcab08d5f63e"
-      (reference "#PWR06") (unit 1) (value "GND") (footprint "")
-    )
-    (path "/f24b66b4-45fc-4e7b-bc4d-d13b5ccb77d9/72e34138-c774-410c-8701-aa4752be6c79"
-      (reference "#PWR07") (unit 1) (value "GND") (footprint "")
-    )
-    (path "/f24b66b4-45fc-4e7b-bc4d-d13b5ccb77d9/0388b81b-7bfb-4a23-9444-5dbf72eb6a1d"
-      (reference "C1") (unit 1) (value "22uF") (footprint "Capacitor_SMD:C_0603_1608Metric")
-    )
-    (path "/f24b66b4-45fc-4e7b-bc4d-d13b5ccb77d9/3b43264c-4f36-4eb7-aaf5-1328e808310f"
-      (reference "C2") (unit 1) (value "22uF") (footprint "Capacitor_SMD:C_0603_1608Metric")
-    )
-    (path "/f24b66b4-45fc-4e7b-bc4d-d13b5ccb77d9/00000000-0000-0000-0000-00005834bc4a"
-      (reference "H1") (unit 1) (value "3mm_Mounting_Hole") (footprint "project_footprints:NPTH_3mm_ID")
-    )
-    (path "/f24b66b4-45fc-4e7b-bc4d-d13b5ccb77d9/00000000-0000-0000-0000-00005834bcdf"
-      (reference "H2") (unit 1) (value "3mm_Mounting_Hole") (footprint "project_footprints:NPTH_3mm_ID")
-    )
-    (path "/f24b66b4-45fc-4e7b-bc4d-d13b5ccb77d9/00000000-0000-0000-0000-000058dfc771"
-      (reference "J1") (unit 1) (value "40HAT") (footprint "Connector_PinSocket_2.54mm:PinSocket_2x20_P2.54mm_Vertical")
-    )
-    (path "/f24b66b4-45fc-4e7b-bc4d-d13b5ccb77d9/443629f4-0a2d-41a4-a71e-9e38e1d7d0bb"
-      (reference "J2") (unit 1) (value "Screw_Terminal_01x02") (footprint "TerminalBlock:TerminalBlock_bornier-2_P5.08mm")
-    )
-    (path "/f24b66b4-45fc-4e7b-bc4d-d13b5ccb77d9/265ee3c7-64fd-410d-98ad-647bd91646d4"
-      (reference "J3") (unit 1) (value "Conn_02x02_Odd_Even") (footprint "Connector_PinHeader_2.54mm:PinHeader_2x02_P2.54mm_Vertical")
-    )
-    (path "/f24b66b4-45fc-4e7b-bc4d-d13b5ccb77d9/643e12dc-0aee-40d2-af28-3b74879d620a"
-      (reference "J4") (unit 1) (value "Conn_02x02_Odd_Even") (footprint "Connector_PinHeader_2.54mm:PinHeader_2x02_P2.54mm_Vertical")
-    )
-    (path "/f24b66b4-45fc-4e7b-bc4d-d13b5ccb77d9/6d47ebf6-9e3b-4e6c-b25b-c7d90bb5c9cd"
-      (reference "J5") (unit 1) (value "Conn_01x08_Male") (footprint "Connector_PinHeader_2.54mm:PinHeader_1x08_P2.54mm_Vertical")
-    )
-    (path "/f24b66b4-45fc-4e7b-bc4d-d13b5ccb77d9/35d30085-edb0-4f16-ad89-187e5980f49d"
-      (reference "J6") (unit 1) (value "Conn_01x08_Male") (footprint "Connector_PinHeader_2.54mm:PinHeader_1x08_P2.54mm_Vertical")
-    )
-    (path "/f24b66b4-45fc-4e7b-bc4d-d13b5ccb77d9/306ce6b9-f963-4bef-a467-1f026a7c8ee3"
-      (reference "J7") (unit 1) (value "Conn_01x03_Male") (footprint "Connector_PinHeader_2.54mm:PinHeader_1x03_P2.54mm_Vertical")
-    )
-    (path "/f24b66b4-45fc-4e7b-bc4d-d13b5ccb77d9/d477b005-312c-49d6-9daa-9d09f8b1b229"
-      (reference "J8") (unit 1) (value "Conn_02x03_Odd_Even") (footprint "Connector_PinHeader_2.54mm:PinHeader_2x03_P2.54mm_Vertical")
-    )
-    (path "/f24b66b4-45fc-4e7b-bc4d-d13b5ccb77d9/00000000-0000-0000-0000-000058e14eb1"
-      (reference "Q1") (unit 1) (value "DMG2305UX") (footprint "Package_TO_SOT_SMD:SOT-23")
-    )
-    (path "/f24b66b4-45fc-4e7b-bc4d-d13b5ccb77d9/4fe2d927-f6b5-4b25-baf3-fe0d2f580488"
-      (reference "Q2") (unit 1) (value "MMDT5401") (footprint "Package_TO_SOT_SMD:SOT-363_SC-70-6")
-    )
-    (path "/f24b66b4-45fc-4e7b-bc4d-d13b5ccb77d9/91d1019a-636c-457d-ad8f-da685ce6ba0f"
-      (reference "Q2") (unit 2) (value "MMDT5401") (footprint "Package_TO_SOT_SMD:SOT-363_SC-70-6")
-    )
-    (path "/f24b66b4-45fc-4e7b-bc4d-d13b5ccb77d9/00000000-0000-0000-0000-000058e15896"
-      (reference "R1") (unit 1) (value "10K") (footprint "Resistor_SMD:R_0603_1608Metric")
-    )
-    (path "/f24b66b4-45fc-4e7b-bc4d-d13b5ccb77d9/00000000-0000-0000-0000-000058e158a1"
-      (reference "R2") (unit 1) (value "47K") (footprint "Resistor_SMD:R_0603_1608Metric")
-    )
-    (path "/f24b66b4-45fc-4e7b-bc4d-d13b5ccb77d9/73a7615d-c086-4c71-bc1d-5d26c31e8c5e"
-      (reference "U1") (unit 1) (value "AMS1117-3.3") (footprint "Package_TO_SOT_SMD:SOT-223-3_TabPin2")
-    )
   )
 )
